File: vocore2-motherboard.sch (EAGLE design)
At the start: 98 parts, among them IC1 AP63205, IC2 FE1.1S, IC3 LM3671MF-3.3, IC4 LM3671MF-3.3, IC5 LM3671MF-3.3, IC7 SN74LVC2G14DBVR, IC8 FT230XS-R, J1 RJHSE-5381, J2 TE_1775470-8, J3 AMPHENOL_1140084168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

Commit message: feat: LED für V_USB
Parts:
- added LED8: RED, led:LEDCHIP-LED0805
- added R22: 330R, rcl:R-EU_R0603
Connections:
- new net N$39: LED8.C, R22.2
- net GND: now also R22.1
- net V_USB: now also LED8.A
Other:
- moved on the sheet: C15, D4, X6
Changed lines of the file:
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@@
 <attribute name="DIGIKEY" value="490-4780-1-ND"/>
 </part>
+<part name="LED8" library="led" library_urn="urn:adsk.eagle:library:259" deviceset="LED" device="CHIP-LED0805" package3d_urn="urn:adsk.eagle:package:15818/2" value="RED">
+<attribute name="DIGIKEY" value="160-1447-1-ND"/>
+</part>
+<part name="GND29" library="supply1" deviceset="GND" device=""/>
+<part name="R22" library="rcl" library_urn="urn:adsk.eagle:library:334" deviceset="R-EU_" device="R0603" package3d_urn="urn:adsk.eagle:package:23555/3" value="330R"/>
 </parts>
 <sheets>
@@
 <attribute name="VALUE" x="237.49" y="33.02" size="1.778" layer="96" rot="MR0"/>
 </instance>
-<instance part="X6" gate="G$1" x="241.3" y="149.86" smashed="yes">
-<attribute name="NAME" x="241.3" y="144.78" size="1.27" layer="95"/>
-</instance>
-<instance part="D4" gate="G$1" x="205.74" y="152.4" smashed="yes" rot="R90">
-<attribute name="FARNELL" x="205.74" y="152.4" size="1.778" layer="96" rot="R90" display="off"/>
-<attribute name="NAME" x="195.58" y="147.2565" size="1.778" layer="95" rot="R90"/>
-<attribute name="VALUE" x="215.8365" y="147.2565" size="1.778" layer="96" rot="R90"/>
-<attribute name="DIGIKEY" x="205.74" y="152.4" size="1.778" layer="96" rot="R90" display="off"/>
-</instance>
-<instance part="C15" gate="G$1" x="185.42" y="154.94" smashed="yes">
-<attribute name="BUERKLIN" x="185.42" y="154.94" size="1.778" layer="96" display="off"/>
-<attribute name="MBM" x="185.42" y="154.94" size="1.778" layer="96" display="off"/>
-<attribute name="PREIS" x="185.42" y="154.94" size="1.778" layer="96" display="off"/>
-<attribute name="NAME" x="186.944" y="155.321" size="1.778" layer="95"/>
-<attribute name="VALUE" x="186.944" y="150.241" size="1.778" layer="96"/>
-</instance>
-<instance part="GND26" gate="1" x="198.12" y="139.7" smashed="yes">
-<attribute name="VALUE" x="195.58" y="137.16" size="1.778" layer="96"/>
-</instance>
-<instance part="GND27" gate="1" x="185.42" y="139.7" smashed="yes">
-<attribute name="VALUE" x="182.88" y="137.16" size="1.778" layer="96"/>
-</instance>
-<instance part="GND28" gate="1" x="236.22" y="144.78" smashed="yes">
-<attribute name="VALUE" x="233.68" y="142.24" size="1.778" layer="96"/>
+<instance part="X6" gate="G$1" x="246.38" y="149.86" smashed="yes">
+<attribute name="NAME" x="246.38" y="144.78" size="1.27" layer="95"/>
+</instance>
+<instance part="D4" gate="G$1" x="210.82" y="152.4" smashed="yes" rot="R90">
+<attribute name="FARNELL" x="210.82" y="152.4" size="1.778" layer="96" rot="R90" display="off"/>
+<attribute name="NAME" x="200.66" y="147.2565" size="1.778" layer="95" rot="R90"/>
+<attribute name="VALUE" x="220.9165" y="147.2565" size="1.778" layer="96" rot="R90"/>
+<attribute name="DIGIKEY" x="210.82" y="152.4" size="1.778" layer="96" rot="R90" display="off"/>
+</instance>
+<instance part="C15" gate="G$1" x="190.5" y="154.94" smashed="yes">
+<attribute name="BUERKLIN" x="190.5" y="154.94" size="1.778" layer="96" display="off"/>
+<attribute name="MBM" x="190.5" y="154.94" size="1.778" layer="96" display="off"/>
+<attribute name="PREIS" x="190.5" y="154.94" size="1.778" layer="96" display="off"/>
+<attribute name="NAME" x="192.024" y="155.321" size="1.778" layer="95"/>
+<attribute name="VALUE" x="192.024" y="150.241" size="1.778" layer="96"/>
+</instance>
+<instance part="GND26" gate="1" x="203.2" y="139.7" smashed="yes">
+<attribute name="VALUE" x="200.66" y="137.16" size="1.778" layer="96"/>
+</instance>
+<instance part="GND27" gate="1" x="190.5" y="139.7" smashed="yes">
+<attribute name="VALUE" x="187.96" y="137.16" size="1.778" layer="96"/>
+</instance>
+<instance part="GND28" gate="1" x="241.3" y="144.78" smashed="yes">
+<attribute name="VALUE" x="238.76" y="142.24" size="1.778" layer="96"/>
 </instance>
 <instance part="GND35" gate="1" x="238.76" y="27.94" smashed="yes" rot="MR0">
@@
 <attribute name="NAME" x="186.182" y="105.1814" size="1.778" layer="95" rot="R180"/>
 <attribute name="VALUE" x="192.024" y="105.1814" size="1.778" layer="96" rot="R180"/>
+</instance>
+<instance part="LED8" gate="G$1" x="170.18" y="157.48" smashed="yes">
+<attribute name="NAME" x="173.736" y="152.908" size="1.778" layer="95" rot="R90"/>
+<attribute name="VALUE" x="175.895" y="152.908" size="1.778" layer="96" rot="R90"/>
+<attribute name="DIGIKEY" x="170.18" y="157.48" size="1.778" layer="96" display="off"/>
+</instance>
+<instance part="GND29" gate="1" x="170.18" y="134.62" smashed="yes">
+<attribute name="VALUE" x="167.64" y="132.08" size="1.778" layer="96"/>
+</instance>
+<instance part="R22" gate="G$1" x="170.18" y="144.78" smashed="yes" rot="R90">
+<attribute name="NAME" x="168.6814" y="140.97" size="1.778" layer="95" rot="R90"/>
+<attribute name="VALUE" x="173.482" y="140.97" size="1.778" layer="96" rot="R90"/>
 </instance>
 </instances>
@@
 </segment>
 <segment>
-<wire x1="198.12" y1="144.78" x2="198.12" y2="142.24" width="0.1524" layer="91"/>
+<wire x1="203.2" y1="144.78" x2="203.2" y2="142.24" width="0.1524" layer="91"/>
 <pinref part="D4" gate="G$1" pin="GND"/>
 <pinref part="GND26" gate="1" pin="GND"/>
@@
 <segment>
 <pinref part="C15" gate="G$1" pin="2"/>
-<wire x1="185.42" y1="142.24" x2="185.42" y2="149.86" width="0.1524" layer="91"/>
+<wire x1="190.5" y1="142.24" x2="190.5" y2="149.86" width="0.1524" layer="91"/>
 <pinref part="GND27" gate="1" pin="GND"/>
 </segment>
 <segment>
 <pinref part="X6" gate="G$1" pin="GND"/>
-<wire x1="238.76" y1="149.86" x2="236.22" y2="149.86" width="0.1524" layer="91"/>
-<wire x1="236.22" y1="149.86" x2="236.22" y2="147.32" width="0.1524" layer="91"/>
+<wire x1="243.84" y1="149.86" x2="241.3" y2="149.86" width="0.1524" layer="91"/>
+<wire x1="241.3" y1="149.86" x2="241.3" y2="147.32" width="0.1524" layer="91"/>
 <pinref part="GND28" gate="1" pin="GND"/>
 </segment>
@@
 <junction x="180.34" y="86.36"/>
 <pinref part="GND43" gate="1" pin="GND"/>
+</segment>
+<segment>
+<pinref part="R22" gate="G$1" pin="1"/>
+<pinref part="GND29" gate="1" pin="GND"/>
+<wire x1="170.18" y1="139.7" x2="170.18" y2="137.16" width="0.1524" layer="91"/>
 </segment>
 </net>
@@
 <segment>
 <pinref part="X6" gate="G$1" pin="D+"/>
-<wire x1="238.76" y1="157.48" x2="236.22" y2="157.48" width="0.1524" layer="91"/>
-<label x="236.22" y="157.48" size="1.27" layer="95" rot="R180" xref="yes"/>
+<wire x1="243.84" y1="157.48" x2="241.3" y2="157.48" width="0.1524" layer="91"/>
+<label x="241.3" y="157.48" size="1.27" layer="95" rot="R180" xref="yes"/>
 </segment>
 <segment>
 <pinref part="D4" gate="G$1" pin="IO1"/>
-<wire x1="213.36" y1="144.78" x2="213.36" y2="142.24" width="0.1524" layer="91"/>
-<wire x1="213.36" y1="142.24" x2="218.44" y2="142.24" width="0.1524" layer="91"/>
-<label x="218.44" y="142.24" size="1.27" layer="95" xref="yes"/>
+<wire x1="218.44" y1="144.78" x2="218.44" y2="142.24" width="0.1524" layer="91"/>
+<wire x1="218.44" y1="142.24" x2="223.52" y2="142.24" width="0.1524" layer="91"/>
+<label x="223.52" y="142.24" size="1.27" layer="95" xref="yes"/>
 </segment>
 <segment>
@@
 <segment>
 <pinref part="X6" gate="G$1" pin="D-"/>
-<wire x1="238.76" y1="154.94" x2="236.22" y2="154.94" width="0.1524" layer="91"/>
-<label x="236.22" y="154.94" size="1.27" layer="95" rot="R180" xref="yes"/>
+<wire x1="243.84" y1="154.94" x2="241.3" y2="154.94" width="0.1524" layer="91"/>
+<label x="241.3" y="154.94" size="1.27" layer="95" rot="R180" xref="yes"/>
 </segment>
 <segment>
 <pinref part="D4" gate="G$1" pin="IO2"/>
-<wire x1="213.36" y1="160.02" x2="213.36" y2="162.56" width="0.1524" layer="91"/>
-<wire x1="213.36" y1="162.56" x2="218.44" y2="162.56" width="0.1524" layer="91"/>
-<label x="218.44" y="162.56" size="1.27" layer="95" xref="yes"/>
+<wire x1="218.44" y1="160.02" x2="218.44" y2="162.56" width="0.1524" layer="91"/>
+<wire x1="218.44" y1="162.56" x2="223.52" y2="162.56" width="0.1524" layer="91"/>
+<label x="223.52" y="162.56" size="1.27" layer="95" xref="yes"/>
 </segment>
 <segment>
@@
 <net name="V_USB" class="0">
 <segment>
-<wire x1="198.12" y1="160.02" x2="198.12" y2="162.56" width="0.1524" layer="91"/>
-<wire x1="198.12" y1="162.56" x2="185.42" y2="162.56" width="0.1524" layer="91"/>
-<label x="182.88" y="162.56" size="1.27" layer="95" rot="R180" xref="yes"/>
+<wire x1="203.2" y1="160.02" x2="203.2" y2="162.56" width="0.1524" layer="91"/>
+<wire x1="203.2" y1="162.56" x2="190.5" y2="162.56" width="0.1524" layer="91"/>
+<label x="187.96" y="162.56" size="1.27" layer="95" rot="R180" xref="yes"/>
 <pinref part="D4" gate="G$1" pin="VCC"/>
-<wire x1="185.42" y1="162.56" x2="182.88" y2="162.56" width="0.1524" layer="91"/>
+<wire x1="190.5" y1="162.56" x2="187.96" y2="162.56" width="0.1524" layer="91"/>
 <pinref part="C15" gate="G$1" pin="1"/>
-<wire x1="185.42" y1="157.48" x2="185.42" y2="162.56" width="0.1524" layer="91"/>
-<junction x="185.42" y="162.56"/>
+<wire x1="190.5" y1="157.48" x2="190.5" y2="162.56" width="0.1524" layer="91"/>
+<junction x="190.5" y="162.56"/>
 </segment>
 <segment>
 <pinref part="X6" gate="G$1" pin="VBUS"/>
-<wire x1="238.76" y1="152.4" x2="236.22" y2="152.4" width="0.1524" layer="91"/>
-<label x="236.22" y="152.4" size="1.27" layer="95" rot="R180" xref="yes"/>
+<wire x1="243.84" y1="152.4" x2="241.3" y2="152.4" width="0.1524" layer="91"/>
+<label x="241.3" y="152.4" size="1.27" layer="95" rot="R180" xref="yes"/>
 </segment>
 <segment>
@@
 <wire x1="165.1" y1="101.6" x2="162.56" y2="101.6" width="0.1524" layer="91"/>
 <label x="162.56" y="101.6" size="1.27" layer="95" rot="R180" xref="yes"/>
+</segment>
+<segment>
+<pinref part="LED8" gate="G$1" pin="A"/>
+<wire x1="170.18" y1="160.02" x2="170.18" y2="162.56" width="0.1524" layer="91"/>
+<label x="170.18" y="162.56" size="1.27" layer="95" rot="R90" xref="yes"/>
 </segment>
 </net>
@@
 </segment>
 </net>
+<net name="N$39" class="0">
+<segment>
+<pinref part="LED8" gate="G$1" pin="C"/>
+<pinref part="R22" gate="G$1" pin="2"/>
+<wire x1="170.18" y1="152.4" x2="170.18" y2="149.86" width="0.1524" layer="91"/>
+</segment>
+</net>

Commit message: feat(brd): threaded inserts for PCIe half-sized card (X3 and X2 only)
Parts:
- X1: value TE_1775838-2 -> TE_1775838-2-FULL; device pachl-con:TE_1775838-2 -> pachl-con:TE_1775838-2-FULL
Changed lines of the file:
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@@
 <attribute name="LCSC" value="C252917"/>
 </part>
-<part name="X1" library="pachl-con" deviceset="TE_1775838-2" device=""/>
+<part name="X1" library="pachl-con" deviceset="TE_1775838-2" device="-FULL" value="TE_1775838-2-FULL"/>
 <part name="IC2" library="Ai_IC" deviceset="FE1.1S" device="">
 <attribute name="SPICEPREFIX" value="X"/>

Commit message: fix: changed led resistor values
Parts:
- R10, R6: value 150R -> 100R
- R2, R4, R5: value 150R -> 470R
Other:
- note added: "I=3mA @ Vf=2V"
Changed lines of the file:
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@@
 </part>
 <part name="GND18" library="supply1" deviceset="GND" device=""/>
-<part name="R2" library="rcl" library_urn="urn:adsk.eagle:library:334" deviceset="R-EU_" device="R0603" package3d_urn="urn:adsk.eagle:package:23555/3" value="150R"/>
+<part name="R2" library="rcl" library_urn="urn:adsk.eagle:library:334" deviceset="R-EU_" device="R0603" package3d_urn="urn:adsk.eagle:package:23555/3" value="470R"/>
 <part name="LED2" library="led" library_urn="urn:adsk.eagle:library:259" deviceset="LED" device="CHIP-LED0805" package3d_urn="urn:adsk.eagle:package:15818/2" value="ORANGE">
 <attribute name="DIGIKEY" value="160-1445-1-ND"/>
 </part>
 <part name="GND19" library="supply1" deviceset="GND" device=""/>
-<part name="R4" library="rcl" library_urn="urn:adsk.eagle:library:334" deviceset="R-EU_" device="R0603" package3d_urn="urn:adsk.eagle:package:23555/3" value="150R"/>
+<part name="R4" library="rcl" library_urn="urn:adsk.eagle:library:334" deviceset="R-EU_" device="R0603" package3d_urn="urn:adsk.eagle:package:23555/3" value="470R"/>
 <part name="LED4" library="led" library_urn="urn:adsk.eagle:library:259" deviceset="LED" device="CHIP-LED0805" package3d_urn="urn:adsk.eagle:package:15818/2" value="ORANGE">
 <attribute name="DIGIKEY" value="160-1445-1-ND"/>
 </part>
 <part name="GND20" library="supply1" deviceset="GND" device=""/>
-<part name="R5" library="rcl" library_urn="urn:adsk.eagle:library:334" deviceset="R-EU_" device="R0603" package3d_urn="urn:adsk.eagle:package:23555/3" value="150R"/>
+<part name="R5" library="rcl" library_urn="urn:adsk.eagle:library:334" deviceset="R-EU_" device="R0603" package3d_urn="urn:adsk.eagle:package:23555/3" value="470R"/>
 <part name="GND21" library="supply1" library_urn="urn:adsk.eagle:library:371" deviceset="GND" device="">
 <attribute name="SPICEPREFIX" value="G"/>
@@
 <attribute name="DIGIKEY" value="160-1446-1-ND"/>
 </part>
-<part name="R6" library="rcl" library_urn="urn:adsk.eagle:library:334" deviceset="R-EU_" device="R0603" package3d_urn="urn:adsk.eagle:package:23555/3" value="150R"/>
+<part name="R6" library="rcl" library_urn="urn:adsk.eagle:library:334" deviceset="R-EU_" device="R0603" package3d_urn="urn:adsk.eagle:package:23555/3" value="100R"/>
 <part name="LED6" library="led" library_urn="urn:adsk.eagle:library:259" deviceset="LED" device="CHIP-LED0805" package3d_urn="urn:adsk.eagle:package:15818/2" value="GREEN">
 <attribute name="DIGIKEY" value="160-1446-1-ND"/>
 </part>
-<part name="R10" library="rcl" library_urn="urn:adsk.eagle:library:334" deviceset="R-EU_" device="R0603" package3d_urn="urn:adsk.eagle:package:23555/3" value="150R"/>
+<part name="R10" library="rcl" library_urn="urn:adsk.eagle:library:334" deviceset="R-EU_" device="R0603" package3d_urn="urn:adsk.eagle:package:23555/3" value="100R"/>
 <part name="LED7" library="led" library_urn="urn:adsk.eagle:library:259" deviceset="LED" device="CHIP-LED0805" package3d_urn="urn:adsk.eagle:package:15818/2" value="GREEN">
 <attribute name="DIGIKEY" value="160-1446-1-ND"/>
@@
 Output</text>
 <text x="22.86" y="25.4" size="1.778" layer="98" rot="R90">I=10mA @ Vf=2V</text>
-<text x="50.8" y="25.4" size="1.778" layer="98" rot="R90">I=10mA @ Vf=2V</text>
+<text x="50.8" y="25.4" size="1.778" layer="98" rot="R90">I=3mA @ Vf=2V</text>
 </plain>
 <instances>
